File: ScreenBoard/ScreenBoard.kicad_pcb (KiCad board)
At the start: 2 copper layers, 25 x 30 mm, 18 parts, among them J1 Conn_01x08_MountingPin, J2 LCD_FPC_0.7mm_welding, Q1 AO3415A, U1 XC6209

Commit message: Fix Error
Parts:
- removed the C1 at (152.7, 86.4)
- removed the C2 at (157.2, 89.6)
- removed the D1 at (154.3, 89.7)
- removed the J1 at (150.2, 81.0)
- removed the J2 at (150.3, 91.1)
- removed the Q1 at (155.5, 92.5)
- removed the R1 at (147.2, 83.9)
- removed the R2 at (149.5, 94.8)
- removed the U1 at (156.1, 86.9)
- added D2: D, Resistor_SMD:R_0603_1608Metric, F.Cu at (137.5, 92.0)
- moved Q1 2.65 mm to (138.6, 94.9)
- moved J2 1.08 mm to (144.0, 91.1)
Connections:
- C2 pad 1: /LCD_BL_VCC -> Net-(C2-Pad1)
- U1 pad 5: /LCD_BL_VCC -> Net-(C2-Pad1)
Routing:
- net GND: track 59.1 -> 3.84 mm, vias 16 -> 32
- net Net-(Q1-Pad1): track 43.6 -> 24.2 mm
- net +3V3: track 26.3 -> 10.9 mm
- net /LCD_SCK: track 20.8 -> 10.1 mm
- net /LCD_MOSI: track 20.8 -> 10.2 mm
- net /RES: track 20.8 -> 10.3 mm
- net +5V: track 20.0 -> 9.50 mm
- net /DC: track 20.4 -> 10.2 mm
- net /LCD_BL_VCC: track 13.4 -> 6.65 mm
- net /LEDA: track 10.4 -> 3.77 mm
- net Net-(J2-Pad8): track 7.60 -> 2.34 mm, vias 1 -> 0
- net Net-(C2-Pad1): track 0.00 -> 4.05 mm
- net /LCD_BL: track 3.78 -> 1.92 mm

Commit message: Fix  Error & add SW
Parts:
- added C3: 100nf, Capacitor_SMD:C_0402_1005Metric, F.Cu at (147.1, 74.8)
- added C4: 100nf, Capacitor_SMD:C_0402_1005Metric, F.Cu at (151.1, 74.8)
- added C5: 100nf, Capacitor_SMD:C_0402_1005Metric, F.Cu at (154.8, 75.2)
- added R3: 5.1k, Capacitor_SMD:C_0402_1005Metric, F.Cu at (148.3, 74.8)
- added R4: 5.1k, Capacitor_SMD:C_0402_1005Metric, F.Cu at (149.8, 74.8)
- added R5: 5.1k, Capacitor_SMD:C_0402_1005Metric, F.Cu at (153.6, 75.3)
- added SW1: C318960, KisonNew:C318960, F.Cu at (138.4, 82.9)
- J1: value Conn_01x08_MountingPin -> Conn_01x12_MountingPin; footprint Connector_FFC-FPC:TE_0-1734839-8_1x08-1MP_P0.5mm_Horizontal -> Connector_FFC-FPC:Hirose_FH12-12S-0.5SH_1x12-1MP_P0.50mm_Horizontal
- Q1: footprint Package_TO_SOT_SMD:SOT-523 -> Package_TO_SOT_SMD:SOT-23
- moved D2 21.8 mm to (144.2, 71.3), turned to 180 degrees
- moved Q1 19.4 mm to (157.0, 88.6), turned to 0 degrees
- moved C2 16.9 mm to (137.7, 72.7), turned to -90 degrees
- moved D1 16.1 mm to (144.1, 73.9), turned to -90 degrees
- moved U1 14.2 mm to (139.9, 72.7), turned to 90 degrees
- moved C1 12.9 mm to (142.6, 73.5), turned to 90 degrees
- moved R2 7.31 mm to (149.7, 88.6), turned to 0 degrees
- moved R1 6.44 mm to (153.8, 87.1), turned to -90 degrees
- moved J1 6.13 mm to (151.2, 79.8), turned to 0 degrees
Connections:
- J1 pad 1: /LCD_BL -> GND
- J1 pad 2: /RES -> /BTN_Down
- J1 pad 3: /LCD_MOSI -> /BTN_Left
- J1 pad 4: /LCD_SCK -> /BTN_Right
- J1 pad 5: /DC -> +5V
- J1 pad 6: GND -> +3V3
- J1 pad 7: +3V3 -> GND
- J1 pad 8: +5V -> /DC
Routing:
- net +3V3: track 10.9 -> 65.8 mm, vias 0 -> 2
- net /BTN_Right: track 0.00 -> 34.2 mm, vias 0 -> 2
- net /BTN_Left: track 0.00 -> 25.7 mm, vias 0 -> 2
- net /LCD_BL_VCC: track 6.65 -> 30.8 mm
- net Net-(Q1-Pad1): track 24.2 -> 2.19 mm
- net /LEDA: track 3.77 -> 20.2 mm
- net /BTN_Down: track 0.00 -> 16.1 mm, vias 0 -> 2
- net Net-(J2-Pad8): track 2.34 -> 13.2 mm
- net /LCD_BL: track 1.92 -> 12.7 mm
- net GND: track 3.84 -> 14.4 mm, vias 32 -> 20
- net /DC: track 10.2 -> 17.5 mm
- net /LCD_SCK: track 10.1 -> 17.1 mm
- net /LCD_MOSI: track 10.2 -> 17.0 mm
- net /RES: track 10.3 -> 17.0 mm
- net +5V: track 9.50 -> 15.8 mm
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Other:
- board text added: "SDCard"
- board text added: "前向"
- board text added: "天线"
- board text removed: "12mm"
- board text removed: "26mm"
- board text removed: "29mm"
- board text removed: "6mm"
