File: ScreenBoard/ScreenBoard.kicad_sch (KiCad schematic)
At the start: 9 parts

Commit message: Fix Error
Parts:
- added D2: D, Resistor_SMD:R_0603_1608Metric, symbol Device:D
- C1, C2: value (none) -> 1uf; footprint (none) -> Capacitor_SMD:C_0402_1005Metric
- D1: value (none) -> D; footprint (none) -> Resistor_SMD:R_0603_1608Metric
- J1: value (none) -> Conn_01x08_MountingPin; footprint (none) -> Connector_FFC-FPC:TE_0-1734839-8_1x08-1MP_P0.5mm_Horizontal
- J2: value (none) -> LCD_FPC_0.7mm_welding; footprint (none) -> KisonNew:FPC_welding_0.7mm_P0.4mm
- Q1: value (none) -> AO3415A; footprint (none) -> Package_TO_SOT_SMD:SOT-523
- R1: value (none) -> 1k; footprint (none) -> Resistor_SMD:R_0402_1005Metric
- R2: value (none) -> 0; footprint (none) -> Resistor_SMD:R_0402_1005Metric
- U1: value (none) -> XC6209; footprint (none) -> Package_TO_SOT_SMD:SOT-23-5
Connections:
- net LCD_BL_VCC: now also D2.1 (K); no longer C2.1, U1.5 (VOUT)
- new net: C2.1, D2.2 (A), U1.5 (VOUT)
Changed lines of the file:
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@@
 (kicad_sch (version 20211123) (generator eeschema)
   (paper "A4")
+  (junction (at 119.888 28.321) (diameter 0) (color 0 0 0 0)
+  )
   (junction (at 92.837 28.321) (diameter 0) (color 0 0 0 0)
   )
@@
     (effects (font (size 1.27 1.27)) (justify right bottom))
   )
-  (label "LCD_BL_VCC" (at 119.888 28.321 0)
+  (label "LCD_BL_VCC" (at 127.508 28.321 0)
     (effects (font (size 1.27 1.27)) (justify left bottom))
   )
@@
     (in_bom yes) (on_board yes)
     (property "Reference" "R2" (id 0) (at 95.758 74.168 90))
-    (property "Value" "" (id 1) (at 100.965 75.565 90))
-    (property "Footprint" "" (id 2) (at 100.965 77.343 90)
+    (property "Value" "0" (id 1) (at 100.965 75.565 90))
+    (property "Footprint" "Resistor_SMD:R_0402_1005Metric" (id 2) (at 100.965 77.343 90)
       (effects (font (size 1.27 1.27)) hide)
     )
@@
     (pin "1")
   )
+  (symbol (lib_id "Device:D") (at 123.698 28.321 180) (unit 1)
+    (in_bom yes) (on_board yes) (fields_autoplaced)
+    (property "Reference" "D2" (id 0) (at 123.698 23.3512 0))
+    (property "Value" "D" (id 1) (at 123.698 25.8881 0))
+    (property "Footprint" "Resistor_SMD:R_0603_1608Metric" (id 2) (at 123.698 28.321 0)
+      (effects (font (size 1.27 1.27)) hide)
+    )
+    (property "Datasheet" "~" (id 3) (at 123.698 28.321 0)
+      (effects (font (size 1.27 1.27)) hide)
+    )
+    (pin "1")
+    (pin "2")
+  )
   (symbol (lib_id "power:GND") (at 104.775 57.785 180) (unit 1)
     (in_bom yes) (on_board yes) (fields_autoplaced)
@@
       (effects (font (size 1.27 1.27)) hide)
     )
-    (property "Value" "" (id 1) (at 104.775 54.2092 0))
+    (property "Value" "GND" (id 1) (at 104.775 54.2092 0))
     (property "Footprint" "" (id 2) (at 104.775 57.785 0)
       (effects (font (size 1.27 1.27)) hide)
@@
       (effects (font (size 1.27 1.27)) hide)
     )
-    (property "Value" "" (id 1) (at 93.9801 75.9988 90)
+    (property "Value" "GND" (id 1) (at 93.9801 75.9988 90)
       (effects (font (size 1.27 1.27)) (justify right))
     )
@@
       (effects (font (size 1.27 1.27)) (justify left))
     )
-    (property "Value" "" (id 1) (at 56.896 75.1717 0)
-      (effects (font (size 1.27 1.27)) (justify left))
-    )
-    (property "Footprint" "" (id 2) (at 56.769 74.676 0)
+    (property "Value" "AO3415A" (id 1) (at 56.896 75.1717 0)
+      (effects (font (size 1.27 1.27)) (justify left))
+    )
+    (property "Footprint" "Package_TO_SOT_SMD:SOT-523" (id 2) (at 56.769 74.676 0)
       (effects (font (size 1.27 1.27)) (justify left) hide)
     )
@@
       (effects (font (size 1.27 1.27)) (justify left))
     )
-    (property "Value" "" (id 1) (at 121.031 73.5207 0)
-      (effects (font (size 1.27 1.27)) (justify left))
-    )
-    (property "Footprint" "" (id 2) (at 109.855 70.485 0)
+    (property "Value" "LCD_FPC_0.7mm_welding" (id 1) (at 121.031 73.5207 0)
+      (effects (font (size 1.27 1.27)) (justify left))
+    )
+    (property "Footprint" "KisonNew:FPC_welding_0.7mm_P0.4mm" (id 2) (at 109.855 70.485 0)
       (effects (font (size 1.27 1.27)) hide)
     )
@@
       (effects (font (size 1.27 1.27)) (justify left))
     )
-    (property "Value" "" (id 1) (at 90.932 35.306 90)
-      (effects (font (size 1.27 1.27)) (justify left))
-    )
-    (property "Footprint" "" (id 2) (at 88.392 30.861 0)
+    (property "Value" "1uf" (id 1) (at 90.932 35.306 90)
+      (effects (font (size 1.27 1.27)) (justify left))
+    )
+    (property "Footprint" "Capacitor_SMD:C_0402_1005Metric" (id 2) (at 88.392 30.861 0)
       (effects (font (size 1.27 1.27)) hide)
     )
@@
       (effects (font (size 1.27 1.27)) (justify left))
     )
-    (property "Value" "" (id 1) (at 122.428 35.306 90)
-      (effects (font (size 1.27 1.27)) (justify left))
-    )
-    (property "Footprint" "" (id 2) (at 119.888 30.861 0)
+    (property "Value" "1uf" (id 1) (at 122.428 35.306 90)
+      (effects (font (size 1.27 1.27)) (justify left))
+    )
+    (property "Footprint" "Capacitor_SMD:C_0402_1005Metric" (id 2) (at 119.888 30.861 0)
       (effects (font (size 1.27 1.27)) hide)
     )
@@
     (in_bom yes) (on_board yes)
     (property "Reference" "R1" (id 0) (at 42.799 68.0552 90))
-    (property "Value" "" (id 1) (at 42.799 72.771 90))
-    (property "Footprint" "" (id 2) (at 42.799 74.549 90)
+    (property "Value" "1k" (id 1) (at 42.799 72.771 90))
+    (property "Footprint" "Resistor_SMD:R_0402_1005Metric" (id 2) (at 42.799 74.549 90)
       (effects (font (size 1.27 1.27)) hide)
     )
@@
       (effects (font (size 1.27 1.27)) (justify left))
     )
-    (property "Value" "" (id 1) (at 42.545 42.291 90)
-      (effects (font (size 1.27 1.27)) (justify left))
-    )
-    (property "Footprint" "" (id 2) (at 35.433 27.686 0)
+    (property "Value" "Conn_01x08_MountingPin" (id 1) (at 42.545 42.291 90)
+      (effects (font (size 1.27 1.27)) (justify left))
+    )
+    (property "Footprint" "Connector_FFC-FPC:TE_0-1734839-8_1x08-1MP_P0.5mm_Horizontal" (id 2) (at 35.433 27.686 0)
       (effects (font (size 1.27 1.27)) hide)
     )
@@
     (in_bom yes) (on_board yes)
     (property "Reference" "U1" (id 0) (at 106.553 21.59 0))
-    (property "Value" "" (id 1) (at 106.553 23.9014 0))
-    (property "Footprint" "" (id 2) (at 106.553 24.511 0)
+    (property "Value" "XC6209" (id 1) (at 106.553 23.9014 0))
+    (property "Footprint" "Package_TO_SOT_SMD:SOT-23-5" (id 2) (at 106.553 24.511 0)
       (effects (font (size 1.27 1.27)) hide)
     )
@@
     (in_bom yes) (on_board yes) (fields_autoplaced)
     (property "Reference" "D1" (id 0) (at 50.165 46.8462 0))
-    (property "Value" "" (id 1) (at 50.165 49.3831 0))
-    (property "Footprint" "" (id 2) (at 50.165 51.816 0)
+    (property "Value" "D" (id 1) (at 50.165 49.3831 0))
+    (property "Footprint" "Resistor_SMD:R_0603_1608Metric" (id 2) (at 50.165 51.816 0)
       (effects (font (size 1.27 1.27)) hide)
     )
@@
       (reference "D1") (unit 1) (value "D") (footprint "Resistor_SMD:R_0603_1608Metric")
     )
+    (path "/158aad19-9736-45f6-b36f-9e02c74763a3"
+      (reference "D2") (unit 1) (value "D") (footprint "Resistor_SMD:R_0603_1608Metric")
+    )
     (path "/d6fb27cf-362d-4568-967c-a5bf49d5931b"

Commit message: Fix  Error & add SW
Parts:
- removed J1: Conn_01x08_MountingPin, Connector_FFC-FPC:TE_0-1734839-8_1x08-1MP_P0.5mm_Horizontal, symbol Connector_Generic_MountingPin:Conn_01x08_MountingPin
- added C3, C4, C5: 100nf, Capacitor_SMD:C_0402_1005Metric, symbol Device:C
- added J1: Conn_01x12_MountingPin, Connector_FFC-FPC:Hirose_FH12-12S-0.5SH_1x12-1MP_P0.50mm_Horizontal, symbol Connector_Generic_MountingPin:Conn_01x12_MountingPin
- added R3, R4, R5: 5.1k, Capacitor_SMD:C_0402_1005Metric, symbol Device:R
- added SW1: C318960, KisonNew:C318960, symbol KisonNew:C318960
- Q1: footprint Package_TO_SOT_SMD:SOT-523 -> Package_TO_SOT_SMD:SOT-23
Connections:
- net +3V3: now also J1.6 (Pin_6), R3.2, R4.2, R5.2
- net +5V: now also J1.5 (Pin_5)
- net DC: now also J1.8 (Pin_8)
- net GND: now also C3.2, C4.2, C5.2, J1.1 (Pin_1), J1.7 (Pin_7), J1.MP (MountPin), SW1.a
- net LCD_BL: now also J1.12 (Pin_12)
- net LCD_MOSI: now also J1.10 (Pin_10)
- net LCD_SCK: now also J1.9 (Pin_9)
- net RES: now also J1.11 (Pin_11)
- new net BTN_Down: C3.1, J1.2 (Pin_2), R3.1, SW1.e
- new net BTN_Left: C4.1, J1.3 (Pin_3), R4.1, SW1.c
- new net BTN_Right: C5.1, J1.4 (Pin_4), R5.1, SW1.f
Other:
- note added: "封装不对，小了"

Commit message: 新款拨轮
Parts:
- removed SW1: C318960, KisonNew:C318960, symbol KisonNew:C318960
- added SW1: C318951, KisonNew:C318951, symbol KisonNew:C318951
Connections:
- net BTN_Down: now also SW1.T
- net BTN_Left: now also SW1.2
- net BTN_Right: now also SW1.1
- net GND: now also SW1.C
Changed lines of the file:
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@@
     (pin "1")
+  )
+  (symbol (lib_id "KisonNew:C318951") (at 180.721 28.829 0) (unit 1)
+    (in_bom yes) (on_board yes) (fields_autoplaced)
+    (property "Reference" "SW1" (id 0) (at 180.3412 19.8983 0))
+    (property "Value" "C318951" (id 1) (at 180.3412 22.4352 0))
+    (property "Footprint" "KisonNew:C318951" (id 2) (at 164.846 24.384 0)
+      (effects (font (size 1.27 1.27)) hide)
+    )
+    (property "Datasheet" "~" (id 3) (at 164.846 24.384 0)
+      (effects (font (size 1.27 1.27)) hide)
+    )
+    (pin "1")
+    (pin "2")
+    (pin "C")
+    (pin "T")
   )
   (symbol (lib_id "power:GND") (at 104.775 57.785 180) (unit 1)
@@
     (pin "2")
   )
-  (symbol (lib_id "KisonNew:C318960") (at 180.721 28.829 0) (unit 1)
-    (in_bom yes) (on_board yes) (fields_autoplaced)
-    (property "Reference" "SW1" (id 0) (at 179.122 19.7205 0))
-    (property "Value" "C318960" (id 1) (at 179.122 22.2574 0))
-    (property "Footprint" "KisonNew:C318960" (id 2) (at 180.721 28.829 0)
-      (effects (font (size 1.27 1.27)) hide)
-    )
-    (property "Datasheet" "~" (id 3) (at 180.721 28.829 0)
-      (effects (font (size 1.27 1.27)) hide)
-    )
-    (pin "a")
-    (pin "c")
-    (pin "e")
-    (pin "f")
-  )
   (symbol (lib_id "power:GND") (at 235.077 30.48 0) (unit 1)
     (in_bom yes) (on_board yes) (fields_autoplaced)
@@
       (reference "R5") (unit 1) (value "5.1k") (footprint "Capacitor_SMD:C_0402_1005Metric")
     )
-    (path "/53f90dd5-3a0b-48eb-965c-6aaa765b9334"
-      (reference "SW1") (unit 1) (value "C318960") (footprint "KisonNew:C318960")
+    (path "/1dbe7728-308d-40ae-b824-b166c49fdb93"
+      (reference "SW1") (unit 1) (value "C318951") (footprint "KisonNew:C318951")
     )
     (path "/e25f0cb2-d101-4680-8039-e28dc3ef0e9b"

Commit message: Fix most 3D parts
Parts:
- J1: footprint Connector_FFC-FPC:Hirose_FH12-12S-0.5SH_1x12-1MP_P0.50mm_Horizontal -> KisonNew:Hirose_FH12-12S-0.5SH_1x12-1MP_P0.50mm_Horizontal
Changed lines of the file:
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@@
       (effects (font (size 1.27 1.27)) (justify left))
     )
-    (property "Footprint" "Connector_FFC-FPC:Hirose_FH12-12S-0.5SH_1x12-1MP_P0.50mm_Horizontal" (id 2) (at 28.575 34.925 0)
+    (property "Footprint" "KisonNew:Hirose_FH12-12S-0.5SH_1x12-1MP_P0.50mm_Horizontal" (id 2) (at 28.575 34.925 0)
       (effects (font (size 1.27 1.27)) hide)
     )
@@
     )
     (path "/483f7aee-8377-41a9-be2e-d078c58ff352"
-      (reference "J1") (unit 1) (value "Conn_01x12_MountingPin") (footprint "Connector_FFC-FPC:Hirose_FH12-12S-0.5SH_1x12-1MP_P0.50mm_Horizontal")
+      (reference "J1") (unit 1) (value "Conn_01x12_MountingPin") (footprint "KisonNew:Hirose_FH12-12S-0.5SH_1x12-1MP_P0.50mm_Horizontal")
     )
     (path "/97181880-94fa-42d4-b759-0e5452e90cce"
